File: tiva_pcb1.sch (KiCad schematic (older format))
At the start: 57 parts, among them K1 CONN_3, P1 CONN_5X2, P2 CONN_5X2, P3 CONN_5X2, P4 MICRO-SD, P5 CONN_2, P6 CONN_3, P7 CONN_4X2, P8 CONN_9, P9 CONN_3X2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

Commit message: First complete version.
Everything routed, DRC passes. Silk screen done, gerbers checked briefly.
Parts:
- removed C15: 100u, symbol CSMALL
- added C15: 100u, symbol CAP
- added R17: 47k, symbol R
- added R18, R19: 0, symbol R
- C6: value 1u -> 10u
- R10, R9: value 0R5 -> 0R22
- R6: value 470 -> 100
Connections:
- net labels added: m_sense1_raw, m_sense2_raw, vboot, vcp, vdcc, vref
- net labels removed: pd7
- wire segments 240 -> 245
Other:
- note added: "0 ohm resistors, connecting TM4C\nanalog input to motor R_sense"
- note added: "R3 and R4\nneed not\nbe fitted"
- moved on the sheet: R2
